Commit message: add gripper tool

File: rtb-data/rtbdata/xacro/ufactory_description/lite6/urdf/lite6.urdf (robot description, URDF)
Before this commit: robot lite6, 8 links, 7 joints
Links:
- added link base
- link link1: geometry collision mesh filename=package://ufactory_description/lite6/meshes/collision/link1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; visual mesh filename=package://ufactory_description/lite6/meshes/visual/link1.stl
- link link2: geometry collision mesh filename=package://ufactory_description/lite6/meshes/collision/link2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; visual mesh filename=package://ufactory_description/lite6/meshes/visual/link2.stl
- link link3: geometry collision mesh filename=package://ufactory_description/lite6/meshes/collision/link3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; visual mesh filename=package://ufactory_description/lite6/meshes/visual/link3.stl
- link link4: geometry collision mesh filename=package://ufactory_description/lite6/meshes/collision/link4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; visual mesh filename=package://ufactory_description/lite6/meshes/visual/link4.stl
- link link5: geometry collision mesh filename=package://ufactory_description/lite6/meshes/collision/link5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; visual mesh filename=package://ufactory_description/lite6/meshes/visual/link5.stl
- link link6: geometry collision mesh filename=package://ufactory_description/lite6/meshes/collision/link6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; visual mesh filename=package://ufactory_description/lite6/meshes/visual/link6.stl
- link link_base: geometry collision mesh filename=package://ufactory_description/lite6/meshes/collision/base.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; visual mesh filename=package://ufactory_description/lite6/meshes/visual/base.stl
- link link_eef: geometry collision mesh filename=package://ufactory_description/lite6/meshes/collision/gripp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; visual mesh filename=package://ufactory_description/lite6/meshes/visual/gripper_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
Joints:
- added joint link_base-base: type fixed, parent link_base, child base, origin xyz=0 0 0 rpy=0 0 0
- joint joint1: limit lower=-2*3.14 upper=2*3.14 effort=50.0 velocity=3.14 -> lower=-6.28318 upper=6.28318 effort=50.0 velocity=3.14
- joint joint4: limit lower=-2*3.14 upper=2*3.14 effort=32.0 velocity=3.14 -> lower=-6.28318 upper=6.28318 effort=32.0 velocity=3.14
- joint joint6: limit lower=-2*3.14 upper=2*3.14 effort=20.0 velocity=3.14 -> lower=-6.28318 upper=6.28318 effort=20.0 velocity=3.14

File: rtb-data/rtbdata/xacro/ufactory_description/lite6/urdf/lite6.urdf.xacro (robot description, xacro)
@@ -1,11 +1,12 @@
 <?xml version="1.0" encoding='utf-8'?>
 <robot xmlns:xacro="http://ros.org/wiki/xacro" name="lite6">
-  <xacro:macro name="lite6_urdf" params="prefix
-    joint1_lower_limit:=${-2.0*pi}  joint1_upper_limit:=${2.0*pi}
-    joint2_lower_limit:=${-2.61799}  joint2_upper_limit:=${2.61799}
-    joint3_lower_limit:=${-0.061087}  joint3_upper_limit:=${5.235988}
-    joint4_lower_limit:=${-2.0*pi}  joint4_upper_limit:=${2.0*pi}
-    joint5_lower_limit:=${-2.1642}  joint5_upper_limit:=${2.1642}
-    joint6_lower_limit:=${-2.0*pi}  joint6_upper_limit:=${2.0*pi}"
+	<xacro:property name="pi" value="3.14159" />
+	<xacro:macro name="lite6" params="prefix
+		joint1_lower_limit  joint1_upper_limit
+		joint2_lower_limit  joint2_upper_limit
+		joint3_lower_limit  joint3_upper_limit
+		joint4_lower_limit  joint4_upper_limit
+		joint5_lower_limit  joint5_upper_limit
+		joint6_lower_limit  joint6_upper_limit"
     >
     <material name="${prefix}White">
@@ -19,5 +20,5 @@
         <origin
           xyz="-0.00829544579053192 3.26357432323433E-05 0.0631194584987089"
-          rpy="0 0 0" />
+          rpy="0 0 ${pi/2}" />
         <mass
           value="1.65393501783165" />
@@ -44,5 +45,5 @@
           rpy="0 0 0" />
         <geometry>
-          <mesh filename="package://ufactory_description/lite6/meshes/visual/base.stl"/>
+          <mesh filename="package://ufactory_description/lite6/meshes/collision/base.stl"/>
         </geometry>
       </collision>
@@ -77,5 +78,5 @@
           rpy="0 0 0" />
         <geometry>
-          <mesh filename="package://ufactory_description/lite6/meshes/visual/link1.stl"/>
+          <mesh filename="package://ufactory_description/lite6/meshes/collision/link1.stl"/>
         </geometry>
       </collision>
@@ -127,5 +128,5 @@
           rpy="0 0 0" />
         <geometry>
-           <mesh filename="package://ufactory_description/lite6/meshes/visual/link2.stl"/>
+           <mesh filename="package://ufactory_description/lite6/meshes/collision/link2.stl"/>
         </geometry>
       </collision>
@@ -177,5 +178,5 @@
           rpy="0 0 0" />
         <geometry>
-           <mesh filename="package://ufactory_description/lite6/meshes/visual/link3.stl"/>
+           <mesh filename="package://ufactory_description/lite6/meshes/collision/link3.stl"/>
         </geometry>
       </collision>
@@ -227,5 +228,5 @@
           rpy="0 0 0" />
         <geometry>
-           <mesh filename="package://ufactory_description/lite6/meshes/visual/link4.stl"/>
+           <mesh filename="package://ufactory_description/lite6/meshes/collision/link4.stl"/>
         </geometry>
       </collision>
@@ -277,5 +278,5 @@
           rpy="0 0 0" />
         <geometry>
-           <mesh filename="package://ufactory_description/lite6/meshes/visual/link5.stl"/>
+           <mesh filename="package://ufactory_description/lite6/meshes/collision/link5.stl"/>
         </geometry>
       </collision>
@@ -327,5 +328,5 @@
           rpy="0 0 0" />
         <geometry>
-           <mesh filename="package://ufactory_description/lite6/meshes/visual/link6.stl"/>
+           <mesh filename="package://ufactory_description/lite6/meshes/collision/link6.stl"/>
         </geometry>
       </collision>
@@ -348,5 +349,37 @@
       <dynamics damping="1.0" friction="1.0"/>
     </joint>
-    <link name="${prefix}link_eef" />
+    <link name="link_eef">
+    <inertial>
+        <origin
+          xyz="0.0 0 0"
+          rpy="0 0 0" />
+        <mass
+          value="0.180" />
+        <inertia
+          ixx="7.726E-05"
+          ixy="1E-06"
+          ixz="4E-07"
+          iyy="8.5665E-05"
+          iyz="-6E-07"
+          izz="1.4814E-04" />
+      </inertial>
+      <visual>
+        <origin
+          xyz="0 0 0"
+          rpy="0 0 0" />
+        <geometry>
+          <mesh filename="package://ufactory_description/lite6/meshes/visual/gripper_lite.stl"/>
+        </geometry>
+        <material name="Silver" />
+      </visual>
+      <collision>
+        <origin
+          xyz="0 0 0"
+          rpy="0 0 0" />
+        <geometry>
+          <mesh filename="package://ufactory_description/lite6/meshes/collision/gripper_lite.stl"/>
+        </geometry>
+      </collision>
+    </link>
     <joint
       name="${prefix}joint_eef"
@@ -360,5 +393,12 @@
         link="${prefix}link_eef" />
     </joint>
+    <!-- ROS link_base to ABB World Coordinates transform -->
+    <link name="${prefix}base" />
+    <joint name="${prefix}link_base-base" type="fixed">
+      <origin xyz="0 0 0" rpy="0 0 0"/>
+      <parent link="${prefix}link_base"/>
+      <child link="${prefix}base"/>
+    </joint>
   </xacro:macro>
-  <xacro:lite6_urdf prefix=""/>
+  <!--<xacro:lite6_urdf prefix=""/> -->
 </robot>

Commit message: urdf path change

File: rtb-data/rtbdata/xacro/ufactory_description/lite6/urdf/lite6.urdf (robot description, URDF)
Before this commit: robot lite6, 9 links, 8 joints
Links:
- link link1: geometry collision mesh filename=package://lite6/meshes/collision/link1.stl; visual mesh filename=package://lite6/meshes/visual/link1.stl
- link link2: geometry collision mesh filename=package://lite6/meshes/collision/link2.stl; visual mesh filename=package://lite6/meshes/visual/link2.stl
- link link3: geometry collision mesh filename=package://lite6/meshes/collision/link3.stl; visual mesh filename=package://lite6/meshes/visual/link3.stl
- link link4: geometry collision mesh filename=package://lite6/meshes/collision/link4.stl; visual mesh filename=package://lite6/meshes/visual/link4.stl
- link link5: geometry collision mesh filename=package://lite6/meshes/collision/link5.stl; visual mesh filename=package://lite6/meshes/visual/link5.stl
- link link6: geometry collision mesh filename=package://lite6/meshes/collision/link6.stl; visual mesh filename=package://lite6/meshes/visual/link6.stl
- link link_base: geometry collision mesh filename=package://lite6/meshes/collision/base.stl; visual mesh filename=package://lite6/meshes/visual/base.stl
- link link_eef: geometry collision mesh filename=package://lite6/meshes/collision/gripper_lite.stl; visual mesh filename=package://lite6/meshes/visual/gripper_lite.stl

File: rtb-data/rtbdata/xacro/ufactory_description/lite6/urdf/lite6.urdf.xacro (robot description, xacro)
@@ -36,14 +36,14 @@
           rpy="0 0 0" />
         <geometry>
-          <mesh filename="package://ufactory_description/lite6/meshes/visual/base.stl"/>
-        </geometry>
-        <material name="${prefix}White" />
-      </visual>
-      <collision>
-        <origin
-          xyz="0 0 0"
-          rpy="0 0 0" />
-        <geometry>
-          <mesh filename="package://ufactory_description/lite6/meshes/collision/base.stl"/>
+          <mesh filename="package://lite6/meshes/visual/base.stl"/>
+        </geometry>
+        <material name="${prefix}White" />
+      </visual>
+      <collision>
+        <origin
+          xyz="0 0 0"
+          rpy="0 0 0" />
+        <geometry>
+          <mesh filename="package://lite6/meshes/collision/base.stl"/>
         </geometry>
       </collision>
@@ -69,14 +69,14 @@
           rpy="0 0 0" />
         <geometry>
-          <mesh filename="package://ufactory_description/lite6/meshes/visual/link1.stl"/>
-        </geometry>
-        <material name="${prefix}White" />
-      </visual>
-      <collision>
-        <origin
-          xyz="0 0 0"
-          rpy="0 0 0" />
-        <geometry>
-          <mesh filename="package://ufactory_description/lite6/meshes/collision/link1.stl"/>
+          <mesh filename="package://lite6/meshes/visual/link1.stl"/>
+        </geometry>
+        <material name="${prefix}White" />
+      </visual>
+      <collision>
+        <origin
+          xyz="0 0 0"
+          rpy="0 0 0" />
+        <geometry>
+          <mesh filename="package://lite6/meshes/collision/link1.stl"/>
         </geometry>
       </collision>
@@ -119,14 +119,14 @@
           rpy="0 0 0" />
         <geometry>
-           <mesh filename="package://ufactory_description/lite6/meshes/visual/link2.stl"/>
-        </geometry>
-        <material name="${prefix}White" />
-      </visual>
-      <collision>
-        <origin
-          xyz="0 0 0"
-          rpy="0 0 0" />
-        <geometry>
-           <mesh filename="package://ufactory_description/lite6/meshes/collision/link2.stl"/>
+           <mesh filename="package://lite6/meshes/visual/link2.stl"/>
+        </geometry>
+        <material name="${prefix}White" />
+      </visual>
+      <collision>
+        <origin
+          xyz="0 0 0"
+          rpy="0 0 0" />
+        <geometry>
+           <mesh filename="package://lite6/meshes/collision/link2.stl"/>
         </geometry>
       </collision>
@@ -169,14 +169,14 @@
           rpy="0 0 0" />
         <geometry>
-           <mesh filename="package://ufactory_description/lite6/meshes/visual/link3.stl"/>
-        </geometry>
-        <material name="${prefix}White" />
-      </visual>
-      <collision>
-        <origin
-          xyz="0 0 0"
-          rpy="0 0 0" />
-        <geometry>
-           <mesh filename="package://ufactory_description/lite6/meshes/collision/link3.stl"/>
+           <mesh filename="package://lite6/meshes/visual/link3.stl"/>
+        </geometry>
+        <material name="${prefix}White" />
+      </visual>
+      <collision>
+        <origin
+          xyz="0 0 0"
+          rpy="0 0 0" />
+        <geometry>
+           <mesh filename="package://lite6/meshes/collision/link3.stl"/>
         </geometry>
       </collision>
@@ -219,14 +219,14 @@
           rpy="0 0 0" />
         <geometry>
-           <mesh filename="package://ufactory_description/lite6/meshes/visual/link4.stl"/>
-        </geometry>
-        <material name="${prefix}White" />
-      </visual>
-      <collision>
-        <origin
-          xyz="0 0 0"
-          rpy="0 0 0" />
-        <geometry>
-           <mesh filename="package://ufactory_description/lite6/meshes/collision/link4.stl"/>
+           <mesh filename="package://lite6/meshes/visual/link4.stl"/>
+        </geometry>
+        <material name="${prefix}White" />
+      </visual>
+      <collision>
+        <origin
+          xyz="0 0 0"
+          rpy="0 0 0" />
+        <geometry>
+           <mesh filename="package://lite6/meshes/collision/link4.stl"/>
         </geometry>
       </collision>
@@ -269,14 +269,14 @@
           rpy="0 0 0" />
         <geometry>
-           <mesh filename="package://ufactory_description/lite6/meshes/visual/link5.stl"/>
-        </geometry>
-        <material name="${prefix}White" />
-      </visual>
-      <collision>
-        <origin
-          xyz="0 0 0"
-          rpy="0 0 0" />
-        <geometry>
-           <mesh filename="package://ufactory_description/lite6/meshes/collision/link5.stl"/>
+           <mesh filename="package://lite6/meshes/visual/link5.stl"/>
+        </geometry>
+        <material name="${prefix}White" />
+      </visual>
+      <collision>
+        <origin
+          xyz="0 0 0"
+          rpy="0 0 0" />
+        <geometry>
+           <mesh filename="package://lite6/meshes/collision/link5.stl"/>
         </geometry>
       </collision>
@@ -319,5 +319,5 @@
           rpy="0 0 0" />
         <geometry>
-           <mesh filename="package://ufactory_description/lite6/meshes/visual/link6.stl"/>
+           <mesh filename="package://lite6/meshes/visual/link6.stl"/>
         </geometry>
         <material name="${prefix}Silver" />
@@ -328,5 +328,5 @@
           rpy="0 0 0" />
         <geometry>
-           <mesh filename="package://ufactory_description/lite6/meshes/collision/link6.stl"/>
+           <mesh filename="package://lite6/meshes/collision/link6.stl"/>
         </geometry>
       </collision>
@@ -369,5 +369,5 @@
           rpy="0 0 0" />
         <geometry>
-          <mesh filename="package://ufactory_description/lite6/meshes/visual/gripper_lite.stl"/>
+          <mesh filename="package://lite6/meshes/visual/gripper_lite.stl"/>
         </geometry>
         <material name="Silver" />
@@ -378,5 +378,5 @@
           rpy="0 0 0" />
         <geometry>
-          <mesh filename="package://ufactory_description/lite6/meshes/collision/gripper_lite.stl"/>
+          <mesh filename="package://lite6/meshes/collision/gripper_lite.stl"/>
         </geometry>
       </collision>

Commit message: path correction

File: rtb-data/rtbdata/xacro/ufactory_description/lite6/urdf/lite6.urdf (robot description, URDF)
Before this commit: robot lite6, 9 links, 8 joints
Links:
- link link1: geometry collision mesh filename=../meshes/collision/link1.stl; visual mesh filename=../meshes/visual/link1.stl
- link link2: geometry collision mesh filename=../meshes/collision/link2.stl; visual mesh filename=../meshes/visual/link2.stl
- link link3: geometry collision mesh filename=../meshes/collision/link3.stl; visual mesh filename=../meshes/visual/link3.stl
- link link4: geometry collision mesh filename=../meshes/collision/link4.stl; visual mesh filename=../meshes/visual/link4.stl
- link link5: geometry collision mesh filename=../meshes/collision/link5.stl; visual mesh filename=../meshes/visual/link5.stl
- link link6: geometry collision mesh filename=../meshes/collision/link6.stl; visual mesh filename=../meshes/visual/link6.stl
- link link_base: geometry collision mesh filename=../meshes/collision/base.stl; visual mesh filename=../meshes/visual/base.stl
- link link_eef: geometry collision mesh filename=../meshes/collision/gripper_lite.stl; visual mesh filename=../meshes/visual/gripper_lite.stl

File: rtb-data/rtbdata/xacro/ufactory_description/lite6/urdf/lite6.urdf.xacro (robot description, xacro)
@@ -36,14 +36,14 @@
           rpy="0 0 0" />
         <geometry>
-          <mesh filename="package://lite6/meshes/visual/base.stl"/>
-        </geometry>
-        <material name="${prefix}White" />
-      </visual>
-      <collision>
-        <origin
-          xyz="0 0 0"
-          rpy="0 0 0" />
-        <geometry>
-          <mesh filename="package://lite6/meshes/collision/base.stl"/>
+          <mesh filename="../meshes/visual/base.stl"/>
+        </geometry>
+        <material name="${prefix}White" />
+      </visual>
+      <collision>
+        <origin
+          xyz="0 0 0"
+          rpy="0 0 0" />
+        <geometry>
+          <mesh filename="../meshes/collision/base.stl"/>
         </geometry>
       </collision>
@@ -69,14 +69,14 @@
           rpy="0 0 0" />
         <geometry>
-          <mesh filename="package://lite6/meshes/visual/link1.stl"/>
-        </geometry>
-        <material name="${prefix}White" />
-      </visual>
-      <collision>
-        <origin
-          xyz="0 0 0"
-          rpy="0 0 0" />
-        <geometry>
-          <mesh filename="package://lite6/meshes/collision/link1.stl"/>
+          <mesh filename="../meshes/visual/link1.stl"/>
+        </geometry>
+        <material name="${prefix}White" />
+      </visual>
+      <collision>
+        <origin
+          xyz="0 0 0"
+          rpy="0 0 0" />
+        <geometry>
+          <mesh filename="../meshes/collision/link1.stl"/>
         </geometry>
       </collision>
@@ -119,14 +119,14 @@
           rpy="0 0 0" />
         <geometry>
-           <mesh filename="package://lite6/meshes/visual/link2.stl"/>
-        </geometry>
-        <material name="${prefix}White" />
-      </visual>
-      <collision>
-        <origin
-          xyz="0 0 0"
-          rpy="0 0 0" />
-        <geometry>
-           <mesh filename="package://lite6/meshes/collision/link2.stl"/>
+           <mesh filename="../meshes/visual/link2.stl"/>
+        </geometry>
+        <material name="${prefix}White" />
+      </visual>
+      <collision>
+        <origin
+          xyz="0 0 0"
+          rpy="0 0 0" />
+        <geometry>
+           <mesh filename="../meshes/collision/link2.stl"/>
         </geometry>
       </collision>
@@ -169,14 +169,14 @@
           rpy="0 0 0" />
         <geometry>
-           <mesh filename="package://lite6/meshes/visual/link3.stl"/>
-        </geometry>
-        <material name="${prefix}White" />
-      </visual>
-      <collision>
-        <origin
-          xyz="0 0 0"
-          rpy="0 0 0" />
-        <geometry>
-           <mesh filename="package://lite6/meshes/collision/link3.stl"/>
+           <mesh filename="../meshes/visual/link3.stl"/>
+        </geometry>
+        <material name="${prefix}White" />
+      </visual>
+      <collision>
+        <origin
+          xyz="0 0 0"
+          rpy="0 0 0" />
+        <geometry>
+           <mesh filename="../meshes/collision/link3.stl"/>
         </geometry>
       </collision>
@@ -219,14 +219,14 @@
           rpy="0 0 0" />
         <geometry>
-           <mesh filename="package://lite6/meshes/visual/link4.stl"/>
-        </geometry>
-        <material name="${prefix}White" />
-      </visual>
-      <collision>
-        <origin
-          xyz="0 0 0"
-          rpy="0 0 0" />
-        <geometry>
-           <mesh filename="package://lite6/meshes/collision/link4.stl"/>
+           <mesh filename="../meshes/visual/link4.stl"/>
+        </geometry>
+        <material name="${prefix}White" />
+      </visual>
+      <collision>
+        <origin
+          xyz="0 0 0"
+          rpy="0 0 0" />
+        <geometry>
+           <mesh filename="../meshes/collision/link4.stl"/>
         </geometry>
       </collision>
@@ -269,14 +269,14 @@
           rpy="0 0 0" />
         <geometry>
-           <mesh filename="package://lite6/meshes/visual/link5.stl"/>
-        </geometry>
-        <material name="${prefix}White" />
-      </visual>
-      <collision>
-        <origin
-          xyz="0 0 0"
-          rpy="0 0 0" />
-        <geometry>
-           <mesh filename="package://lite6/meshes/collision/link5.stl"/>
+           <mesh filename="../meshes/visual/link5.stl"/>
+        </geometry>
+        <material name="${prefix}White" />
+      </visual>
+      <collision>
+        <origin
+          xyz="0 0 0"
+          rpy="0 0 0" />
+        <geometry>
+           <mesh filename="../meshes/collision/link5.stl"/>
         </geometry>
       </collision>
@@ -319,5 +319,5 @@
           rpy="0 0 0" />
         <geometry>
-           <mesh filename="package://lite6/meshes/visual/link6.stl"/>
+           <mesh filename="../meshes/visual/link6.stl"/>
         </geometry>
         <material name="${prefix}Silver" />
@@ -328,5 +328,5 @@
           rpy="0 0 0" />
         <geometry>
-           <mesh filename="package://lite6/meshes/collision/link6.stl"/>
+           <mesh filename="../meshes/collision/link6.stl"/>
         </geometry>
       </collision>
@@ -369,5 +369,5 @@
           rpy="0 0 0" />
         <geometry>
-          <mesh filename="package://lite6/meshes/visual/gripper_lite.stl"/>
+          <mesh filename="../meshes/visual/gripper_lite.stl"/>
         </geometry>
         <material name="Silver" />
@@ -378,5 +378,5 @@
           rpy="0 0 0" />
         <geometry>
-          <mesh filename="package://lite6/meshes/collision/gripper_lite.stl"/>
+          <mesh filename="../meshes/collision/gripper_lite.stl"/>
         </geometry>
       </collision>
