Commit message: mycobot fix

File: rtb-data/rtbdata/xacro/elephant_robotics/mycobot_280_pi/urdf/mycobot_280_pi.urdf (robot description, URDF)
Before this commit: robot firefighter, 8 links, 7 joints
Joints:
- joint g_base_to_joint1: axis 0 0 0 -> 0 0 1; type fixed -> revolute
- joint joint6output_to_joint6: type revolute -> fixed
